Commit message: Edits to better align with usma_gvrbot
Edits as a result from troubleshooting transition from Gazebo to teleop Cartographer.

File: jackal_description/urdf/jackal_orig.urdf.xacro (robot description, xacro)
@@ -1,7 +1,4 @@
 <?xml version="1.0"?>
 <robot name="jackal" xmlns:xacro="http://www.ros.org/wiki/xacro">
-  <!-- -->
-  <xacro:include filename="$(find sara_description)/urdf/sara.urdf.xacro"/>
-  <xacro:include filename="$(find jackal_description)/urdf/inertial_tensors.urdf.xacro"/>
   <xacro:property name="PI" value="3.1415926535897931" />
   <xacro:property name="wheelbase" value="0.262" />
@@ -113,6 +110,4 @@
         izz="0.4485"/>
       </inertial>
-      <parent link="base_link"/>
-      <child link="chassis_link" />
   </link>
   <xacro:unless value="$(optenv JACKAL_FRONT_ACCESSORY_FENDER 0)">
@@ -181,5 +176,5 @@
        to supply the joint between it and imu_link. This is important so that imu_link
        always points to the "active" IMU. When an upgrade IMU is connected, the
-       internal_imu_link should remain, but imu_link should point to the upgrade one.
+       internal_imu_link should remain, but imu_link should point to the upgrade one. -->
   <link name="imu_link">
     <inertial>
@@ -192,5 +187,5 @@
     <parent link="chassis_link" />
     <child link="imu_link" />
-  </joint>-->
+  </joint>
   <!-- TODO: Same note as applies to imu_link -->
   <link name="navsat_link">
@@ -234,5 +229,3 @@
   <!-- Optional custom includes. -->
   <xacro:include filename="$(optenv JACKAL_URDF_EXTRAS empty.urdf)" />
-  <!-- -->
-  <xacro:sara parent_link="base_link" version="jackal"/>
 </robot>
