Commit message: start of solution

File: jackal_description/urdf/jackal.urdf.xacro (robot description, xacro)
@@ -181,5 +181,5 @@
        to supply the joint between it and imu_link. This is important so that imu_link
        always points to the "active" IMU. When an upgrade IMU is connected, the
-       internal_imu_link should remain, but imu_link should point to the upgrade one.
+       internal_imu_link should remain, but imu_link should point to the upgrade one. -->
   <link name="imu_link">
     <inertial>
@@ -192,5 +192,5 @@
     <parent link="chassis_link" />
     <child link="imu_link" />
-  </joint>-->
+  </joint>
   <!-- TODO: Same note as applies to imu_link -->
   <link name="navsat_link">

Commit message: Update jackal_description

File: jackal_description/urdf/jackal.urdf.xacro (robot description, xacro)
@@ -113,6 +113,4 @@
         izz="0.4485"/>
       </inertial>
-      <parent link="base_link"/>
-      <child link="chassis_link" />
   </link>
   <xacro:unless value="$(optenv JACKAL_FRONT_ACCESSORY_FENDER 0)">
