Commit message: Add files via upload
Changes to remove redundancy in velodyne macros, link name updates.

File: sara_description/urdf/sara.urdf.xacro (robot description, xacro)
@@ -6,5 +6,7 @@
   <xacro:include filename="$(find ouster_description)/urdf/OS1-64.urdf.xacro"/>
   -->
+  <!--
   <xacro:include filename="$(find velodyne_description)/urdf/VLP-16.urdf.xacro"/>
+  -->
   <xacro:include filename="$(find velodyne_description)/urdf/HDL-32E.urdf.xacro"/>
   <link name="unit_base_link">
@@ -44,12 +46,12 @@
   </joint>
   <!-- NBL: Realsense D435i Link -->
-  <link name="realsense_link"/>
-  <joint name="realsense_joint" type="fixed">
+  <link name="camera_link"/>
+  <joint name="camera_joint" type="fixed">
     <parent link="unit_base_link" />
-    <child link="realsense_link" />
+    <child link="camera_link" />
     <origin xyz="0.140 0 0.194075" rpy="0 0 0" />
   </joint>
-  <xacro:intel_realsense_mount prefix="camera" topic="realsense" parent_link="realsense_link"/>
-  <!-- NBL: Lidar Link (Ouster OS1-64 parameters using Velodyne plugins) -->
+  <xacro:intel_realsense_mount prefix="camera" topic="realsense" parent_link="camera_link"/>
+  <!-- NBL: Lidar Link (Ouster OS1-64 parameters using Velodyne plugins)
   <link name="lidar_link"/>
   <joint name="lidar_joint" type="fixed">
@@ -58,9 +60,12 @@
     <origin xyz="0.0 0 0.335" rpy="0 0 1.5708" />
   </joint>
+  -->
+  <!--
   <xacro:VLP-16 parent="unit_base_link" name="velodyne" topic="/velodyne_points" hz="10" samples="512">
     <origin xyz="0 0 0.335" rpy="0 0 1.5708" />
   </xacro:VLP-16>
+  -->
   <xacro:HDL-32E parent="unit_base_link" name="velodyne2" topic="/velodyne_points2" hz="10" samples="512">
-    <origin xyz="0 0 0.535" rpy="0 0 1.5708" />
+    <origin xyz="0 0 0.335" rpy="0 0 1.5708" />
   </xacro:HDL-32E>
   <!--

File: velodyne_description/urdf/HDL-32E.urdf.xacro (robot description, xacro)
@@ -16,4 +16,10 @@
           izz="${0.5 * 1.0 * (0.04267*0.04267)}"/>
       </inertial>
+      <visual>
+        <origin xyz="0 0 0" rpy="0 0 0" />
+        <geometry>
+          <mesh filename="package://ouster_description/meshes/os1_64.dae" /> <!--package://velodyne_description/meshes/VLP16_base_1.dae" />-->
+        </geometry>
+      </visual>
       <!--
       <visual>

Commit message: Add files via upload
sara and jackal description files on NUC43 as of 12 March, 2021

File: sara_description/urdf/sara.urdf.xacro (robot description, xacro)
@@ -2,10 +2,15 @@
 <robot name="sara" xmlns:xacro="http://www.ros.org/wiki/xacro">
   <xacro:macro name="sara" params="parent_link version">
+  <!--
   <xacro:include filename="$(find sara_description)/urdf/accessories/intel_realsense.urdf.xacro"/>
+  -->
   <!--
   <xacro:include filename="$(find ouster_description)/urdf/OS1-64.urdf.xacro"/>
   -->
+  <!--
+  <xacro:include filename="$(find ouster_description)/urdf/os1_sensor.urdf.xacro"/>
   <xacro:include filename="$(find velodyne_description)/urdf/VLP-16.urdf.xacro"/>
   <xacro:include filename="$(find velodyne_description)/urdf/HDL-32E.urdf.xacro"/>
+  -->
   <link name="unit_base_link">
     <visual>
@@ -43,5 +48,5 @@
     </xacro:if>
   </joint>
-  <!-- NBL: Realsense D435i Link -->
+  <!-- NBL: Realsense D435i Link
   <link name="realsense_link"/>
   <joint name="realsense_joint" type="fixed">
@@ -50,25 +55,30 @@
     <origin xyz="0.140 0 0.194075" rpy="0 0 0" />
   </joint>
-  <xacro:intel_realsense_mount prefix="camera" topic="realsense" parent_link="realsense_link"/>
+  <xacro:intel_realsense_mount prefix="camera" topic="realsense" parent_link="realsense_link"/>-->
   <!-- NBL: Lidar Link (Ouster OS1-64 parameters using Velodyne plugins) -->
-  <link name="lidar_link"/>
-  <joint name="lidar_joint" type="fixed">
+  <link name="os_sensor"/>
+  <joint name="os_sensor_joint" type="fixed">
     <parent link="unit_base_link" />
-    <child link="lidar_link" />
+    <child link="os_sensor" />
     <origin xyz="0.0 0 0.335" rpy="0 0 1.5708" />
   </joint>
+  <!--
+  <xacro:OS1-64 parent="unit_base_link" name="os_sensor" topic_points="/os_cloud_node/points"/>
+  -->
+  <!--
+  <xacro:os1_sensor parent="unit_base_link" name="os1_sensor" topic_points="/os1_cloud_node/points"/>
+    <origin xyz="0 0 0.335" rpy="0 0 0" />
+  </xacro:OS1-64>
+  -->
+  <!--
   <xacro:VLP-16 parent="unit_base_link" name="velodyne" topic="/velodyne_points" hz="10" samples="512">
     <origin xyz="0 0 0.335" rpy="0 0 1.5708" />
   </xacro:VLP-16>
-  <xacro:HDL-32E parent="unit_base_link" name="velodyne2" topic="/velodyne_points2" hz="10" samples="512">
+  <xacro:HDL-32E parent="unit_base_link" name="velodyne2" topic="Microstrain/velodyne_points2" hz="10" samples="512">
     <origin xyz="0 0 0.535" rpy="0 0 1.5708" />
   </xacro:HDL-32E>
-  <!--
-  <xacro:OS1-64 topic_points="os1_cloud_node/points" parent="unit_base_link">
-    <origin xyz="0 0 0.335" rpy="0 0 0" />
-  </xacro:OS1-64>
   -->
   <!-- Microstrain IMU LINK -->
-  <link name="microstrain_link">
+  <link name="imu_link">
     <visual>
       <geometry>
@@ -83,7 +93,7 @@
     </collision>
   </link>
-  <joint name="microstrain_joint" type="fixed">
+  <joint name="imu_joint" type="fixed">
     <parent link="unit_base_link" />
-    <child link="microstrain_link" />
+    <child link="imu_link" />
     <origin xyz="0 0 0.00645" rpy="0 0 0" />
   </joint>

Commit message: working with bagfile

File: sara_description/urdf/sara.urdf.xacro (robot description, xacro)
@@ -61,5 +61,5 @@
     <parent link="unit_base_link" />
     <child link="os_sensor" />
-    <origin xyz="0.0 0 0.335" rpy="0 0 1.5708" />
+    <origin xyz="0.0 0 0.335" rpy="0 0 0" />
   </joint>
   <!--

Commit message: Update sara_description

File: sara_description/urdf/sara.urdf.xacro (robot description, xacro)
@@ -37,5 +37,5 @@
     </xacro:if>
     <xacro:if value="${version == 'jackal'}">
-      <origin xyz="0.10 0 0.213" rpy="0 0 0" />
+      <origin xyz="0.00475 0 0.213" rpy="0 0 0" />
     </xacro:if>
     <xacro:if value="${version == 'gvrbot'}">
